File: hardware/SkillGame.kicad_sch (KiCad schematic)
At the start: 134 parts, among them J1 Conn_01x02_Pin, J2 Conn_02x20_Odd_Even, J3 Conn_01x02_Pin, J4 Conn_01x02_Pin, J5 Conn_01x02_Pin, Q1 PN2222A, Q10 PN2222A, Q11 PN2222A, Q12 PN2222A, Q13 PN2222A, Q14 PN2222A, Q15 PN2222A, Q16 PN2222A, Q17 PN2222A, Q18 PN2222A, Q2 PN2222A, Q3 PN2222A, Q4 PN2222A, Q5 PN2222A, Q6 PN2222A, Q7 TIP120, Q8 TIP120, Q9 PN2222A, SW0 SW_DPST_x2, SW1 SW_DPST_x2, SW10 SW_DPST_x2, SW11 SW_DPST_x2, SW12 SW_DPST_x2, SW13 SW_DPST_x2, SW14 SW_DPST_x2, SW15 SW_DPST_x2, SW16 SW_DPST_x2, SW17 SW_DPST_x2, SW18 SW_DPST_x2, SW19 SW_DPST_x2, SW2 SW_DPST_x2, SW20 SW_DPST_x2, SW21 SW_DPST_x2, SW22 SW_DPST_x2, SW23-1 SW_DPST_x2, SW23-2 SW_DPST_x2, SW23-3 SW_DPST_x2, SW23-4 SW_DPST_x2, SW23-5 SW_DPST_x2, SW23-6 SW_DPST_x2, SW23-7 SW_DPST_x2, SW24 SW_DPST_x2, SW25 SW_DPST_x2, SW26 SW_DPST_x2, SW27 SW_DPST_x2, SW3 SW_DPST_x2, SW4 SW_DPST_x2, SW5 SW_DPST_x2, SW6 SW_DPST_x2, SW7 SW_DPST_x2, SW8 SW_DPST_x2, SW9 SW_DPST_x2, U1 Conn_01x11_Socket_FT232H, U2 Conn_01x11_Socket_FT232H, U3 Conn_01x11_Socket_FT232H, U4 Conn_01x11_Socket_FT232H

Commit message: Show the LED lamps in the schematic; double the 100/200/300/400 holes
- Schematic: added all 16 score-lamp bulbs as #555 wedge LED symbols, with
  the 100/200/300/400 holes drawing TWO bulbs each (parallel, same output)
  for double brightness. Non-polar bulbs; ERC clean.
- The board's lamp resistors R30-R62 are now 0 R links (schematic + PCB) --
  the pre-resistored #555 bulb self-limits and a 6.3 V bulb is safely
  under-driven on the 5 V rail. DRC clean.
- App: the SCORE LAMPS block now shows the LED bulb bank; updated the lamp
  and 5 V-rail text to match (no more 220 ohm).
- BOM + assembly guide: 20 #555 bulbs + 20 sockets, 0 R lamp links, and the
  WezeBull logo on the guide's cover. Sourced BOM total now $477.52.
- README: logo, badges, How-it-plays, Features and Hardware sections.
Parts:
- added D100, D101, D102, D103, D104, D105, D106, D107, D108, D109, D110, D111, D112, D113, D114, D115, D116, D117, D118, D119: 555, symbol Device:LED
- R30, R32, R34, R36, R38, R40, R53, R54, R55, R56, R57, R58, R59, R60, R61, R62: value 220 Ohm -> 0 R
Connections:
- net GNDREF: now also J2.5 (Pin_5), Q3.3 (C), D104.1 (K), D105.1 (K)
- net LP20: now reaches J2.16 (Pin_16), R54.1
- net LP20: now also D111.2 (A)
- net LPWIN: now reaches J2.12 (Pin_12), R40.1
- net LPWIN: now also D109.2 (A)
- net LN50: now reaches J2.21 (Pin_21), Q13.3 (C)
- net LN50: now also D114.1 (K)
- net LP10: now reaches J2.14 (Pin_14), R53.1
- net LP10: now also D110.2 (A)
- net LPGO: now reaches J2.10 (Pin_10), R38.1
- net LPGO: now also D108.2 (A)
- net LN100: now reaches J2.1 (Pin_1), Q1.3 (C)
- net LN100: now also D100.1 (K), D101.1 (K)
- net LP60: now reaches J2.24 (Pin_24), R58.1
- net LP60: now also D115.2 (A)
- net LN30: now reaches J2.17 (Pin_17), Q11.3 (C)
- net LN30: now also D112.1 (K)
- net LPTILT: now reaches J2.32 (Pin_32), R62.1
- net LPTILT: now also D119.2 (A)
- net LNGO: now reaches J2.9 (Pin_9), Q5.3 (C)
- net LNGO: now also D108.1 (K)
- net LP100: now reaches J2.2 (Pin_2), R30.1
- net LP100: now also D100.2 (A), D101.2 (A)
- net LNTILT: now reaches J2.31 (Pin_31), Q18.3 (C)
- net LNTILT: now also D119.1 (K)
- net LP70: now reaches J2.26 (Pin_26), R59.1
- net LP70: now also D116.2 (A)
- net LN20: now reaches J2.4 (Pin_4), R32.1
- net LN20: now also J2.15 (Pin_15), J2.6 (Pin_6), Q10.3 (C), R34.1, D102.2 (A), D103.2 (A), D104.2 (A), D105.2 (A), D111.1 (K)
- net LP90: now reaches J2.30 (Pin_30), R61.1
- net LP90: now also D118.2 (A)
- net LN200: now reaches J2.3 (Pin_3), Q2.3 (C)
- net LN200: now also D102.1 (K), D103.1 (K)
- net LNWIN: now reaches J2.11 (Pin_11), Q6.3 (C)
- net LNWIN: now also D109.1 (K)
- net LN10: now reaches J2.13 (Pin_13), Q9.3 (C)
- net LN10: now also D110.1 (K)
- net LP30: now reaches J2.18 (Pin_18), R55.1
- net LP30: now also D112.2 (A)
- net LN40: now reaches J2.19 (Pin_19), Q12.3 (C)
- net LN40: now also D113.1 (K)
- net LP40: now reaches J2.20 (Pin_20), R56.1
- net LP40: now also D113.2 (A)
- net LP50: now reaches J2.22 (Pin_22), R57.1
- net LP50: now also D114.2 (A)
- net LN60: now reaches J2.23 (Pin_23), Q14.3 (C)
- net LN60: now also D115.1 (K)
- net LN70: now reaches J2.25 (Pin_25), Q15.3 (C)
- net LN70: now also D116.1 (K)
- net LN80: now reaches J2.27 (Pin_27), Q16.3 (C)
- net LN80: now also D117.1 (K)
- net LP80: now reaches J2.28 (Pin_28), R60.1
- net LP80: now also D117.2 (A)
- net LN90: now reaches J2.29 (Pin_29), Q17.3 (C)
- net LN90: now also D118.1 (K)
- net LN400: now reaches J2.7 (Pin_7), Q4.3 (C)
- net LN400: now also D106.1 (K), D107.1 (K)
- net LP400: now reaches J2.8 (Pin_8), R36.1
- net LP400: now also D106.2 (A), D107.2 (A)
Other:
- note added: "LAMPS: each pair drives an off-board #555 wedge LED bulb (6.3 V non-polar, self-limiting). R30-R62 = 0 R links (the bulb has its own resistor; the 5 V rail under-drives a 6.3 V bulb = safe). 100 / 200 / 300 / 400 hole = TWO bulbs in parallel on the same J2 output = double brightness."

Commit message: Add 28 switch-input debounce caps (100 nF) to the board
- Schematic: added C1-C28, one 100 nF cap from each switch input to GND,
  in parallel with the 10k pull-down (~1 ms RC debounce + noise filter on
  the long playfield leads). Enlarged the sheet to fit the cap bank. ERC at
  the benign baseline; all 28 netlist-verified across input<->GND.
- PCB: placed all 28 as 0805 SMD on the back, next to each pull-down (GND
  pad on the pour, input to the pull-down). 3D back render updated.
- BOM + guide + app schematic images updated (BOM total now $507.16, guide
  24 pages with a debounce-cap step). Synced to the live OneDrive KiCad.
Parts:
- added C1, C10, C11, C12, C13, C14, C15, C16, C17, C18, C19, C2, C20, C21, C22, C23, C24, C25, C26, C27, C28, C3, C4, C5, C6, C7, C8, C9: 100nF, Capacitor_SMD:C_0805_2012Metric, symbol Device:C
Connections:
- net GNDREF: now also C1.1, C10.1, C10.2, C11.1, C11.2, C12.1, C12.2, C13.1, C14.1, C15.1, C16.1, C17.1, C18.1, C18.2, C19.1, C19.2, C2.1, C20.1, C20.2, C21.1, C21.2, C22.1, C22.2, C23.1, C23.2, C24.1, C24.2, C25.1, C26.1, C27.1, C28.1, C3.1, C4.1, C5.1, C6.1, C6.2, C7.1, C7.2, C8.1, C8.2, C9.1, C9.2
- net SWIN13: now reaches R14.1, SW13.2 (B), U2.9 (D5)
- net SWIN13: now also C14.2
- net SWIN0: now reaches R1.1, SW0.2 (B), U1.8 (D4)
- net SWIN0: now also C1.2
- net SWIN2: now reaches R3.1, SW2.2 (B), U1.10 (D6)
- net SWIN2: now also C3.2
- net SWIN3: now reaches R4.1, SW3.2 (B), U1.11 (D7)
- net SWIN3: now also C4.2
- net SWIN4: now reaches R5.1, SW4.2 (B), U1.12 (C0)
- net SWIN4: now also C5.2
- net SWIN1: now reaches R2.1, SW1.2 (B), U1.9 (D5)
- net SWIN1: now also C2.2
- net SWIN14: now reaches R15.1, SW14.2 (B), U2.10 (D6)
- net SWIN14: now also C15.2
- net SWIN15: now reaches R16.1, SW15.2 (B), U2.11 (D7)
- net SWIN15: now also C16.2
- net SWIN16: now reaches R17.1, SW16.2 (B), U2.12 (C0)
- net SWIN16: now also C17.2
- net SWIN12: now reaches R13.1, SW12.2 (B), U2.8 (D4)
- net SWIN12: now also C13.2
- net SWIN24: now reaches R25.1, SW24.2 (B), U3.8 (D4)
- net SWIN24: now also C25.2
- net SWIN25: now reaches R26.1, SW25.2 (B), U3.9 (D5)
- net SWIN25: now also C26.2
- net SWIN26: now reaches R27.1, SW26.2 (B), U3.10 (D6)
- net SWIN26: now also C27.2
- net SWIN27: now reaches R28.1, SW27.2 (B), U3.11 (D7)
- net SWIN27: now also C28.2
Other:
- note added: "SWITCH-INPUT DEBOUNCE CAPS - 100 nF from each input to GND (with the 10k pull-down = ~1 ms RC)."
