File: hardware/SkillGame.kicad_pcb (KiCad board)
At the start: 2 copper layers, 191 x 112.5 mm, 135 parts, among them J1 Conn_01x02_Pin, J2 Conn_02x20_Odd_Even, J3 Conn_01x02_Pin, J4 Conn_01x02_Pin, J5 Conn_01x02_Pin, Q1 PN2222A, Q10 PN2222A, Q11 PN2222A, Q12 PN2222A, Q13 PN2222A, Q14 PN2222A, Q15 PN2222A, Q16 PN2222A, Q17 PN2222A, Q18 PN2222A, Q2 PN2222A, Q3 PN2222A, Q4 PN2222A, Q5 PN2222A, Q6 PN2222A, Q7 TIP120, Q8 TIP120, Q9 PN2222A, SW0 SW_DPST_x2, SW1 SW_DPST_x2, SW10 SW_DPST_x2, SW11 SW_DPST_x2, SW12 SW_DPST_x2, SW13 SW_DPST_x2, SW14 SW_DPST_x2, SW15 SW_DPST_x2, SW16 SW_DPST_x2, SW17 SW_DPST_x2, SW18 SW_DPST_x2, SW19 SW_DPST_x2, SW2 SW_DPST_x2, SW20 SW_DPST_x2, SW21 SW_DPST_x2, SW22 SW_DPST_x2, SW23-1 SW_DPST_x2, SW23-2 SW_DPST_x2, SW23-3 SW_DPST_x2, SW23-4 SW_DPST_x2, SW23-5 SW_DPST_x2, SW23-6 SW_DPST_x2, SW23-7 SW_DPST_x2, SW24 SW_DPST_x2, SW25 SW_DPST_x2, SW26 SW_DPST_x2, SW27 SW_DPST_x2, SW3 SW_DPST_x2, SW4 SW_DPST_x2, SW5 SW_DPST_x2, SW6 SW_DPST_x2, SW7 SW_DPST_x2, SW8 SW_DPST_x2, SW9 SW_DPST_x2, U1 Conn_01x11_Socket_FT232H, U2 Conn_01x11_Socket_FT232H, U3 Conn_01x11_Socket_FT232H, U4 Conn_01x11_Socket_FT232H

Commit message: Show the LED lamps in the schematic; double the 100/200/300/400 holes
- Schematic: added all 16 score-lamp bulbs as #555 wedge LED symbols, with
  the 100/200/300/400 holes drawing TWO bulbs each (parallel, same output)
  for double brightness. Non-polar bulbs; ERC clean.
- The board's lamp resistors R30-R62 are now 0 R links (schematic + PCB) --
  the pre-resistored #555 bulb self-limits and a 6.3 V bulb is safely
  under-driven on the 5 V rail. DRC clean.
- App: the SCORE LAMPS block now shows the LED bulb bank; updated the lamp
  and 5 V-rail text to match (no more 220 ohm).
- BOM + assembly guide: 20 #555 bulbs + 20 sockets, 0 R lamp links, and the
  WezeBull logo on the guide's cover. Sourced BOM total now $477.52.
- README: logo, badges, How-it-plays, Features and Hardware sections.
Parts:
- R30, R32, R34, R36, R38, R40, R53, R54, R55, R56, R57, R58, R59, R60, R61, R62: value 220 Ohm -> 0 R
Changed lines of the file:
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@@
 			)
 		)
-		(property "Value" "220 Ohm"
+		(property "Value" "0 R"
 			(at 2.54 1.92 0)
 			(layer "F.Fab")
@@
 			)
 		)
-		(property "Value" "220 Ohm"
+		(property "Value" "0 R"
 			(at 2.54 1.92 0)
 			(layer "F.Fab")
@@
 			)
 		)
-		(property "Value" "220 Ohm"
+		(property "Value" "0 R"
 			(at 2.54 1.92 0)
 			(layer "F.Fab")
@@
 			)
 		)
-		(property "Value" "220 Ohm"
+		(property "Value" "0 R"
 			(at 2.54 1.92 0)
 			(layer "F.Fab")
@@
 			)
 		)
-		(property "Value" "220 Ohm"
+		(property "Value" "0 R"
 			(at 2.54 1.92 0)
 			(layer "F.Fab")
@@
 			)
 		)
-		(property "Value" "220 Ohm"
+		(property "Value" "0 R"
 			(at 2.54 1.92 0)
 			(layer "F.Fab")
@@
 			)
 		)
-		(property "Value" "220 Ohm"
+		(property "Value" "0 R"
 			(at 2.54 1.92 0)
 			(layer "F.Fab")
@@
 			)
 		)
-		(property "Value" "220 Ohm"
+		(property "Value" "0 R"
 			(at 2.54 1.92 0)
 			(layer "F.Fab")
@@
 			)
 		)
-		(property "Value" "220 Ohm"
+		(property "Value" "0 R"
 			(at 2.54 1.92 0)
 			(layer "F.Fab")
@@
 			)
 		)
-		(property "Value" "220 Ohm"
+		(property "Value" "0 R"
 			(at 2.54 1.92 0)
 			(layer "F.Fab")
@@
 			)
 		)
-		(property "Value" "220 Ohm"
+		(property "Value" "0 R"
 			(at 2.54 1.92 0)
 			(layer "F.Fab")
@@
 			)
 		)
-		(property "Value" "220 Ohm"
+		(property "Value" "0 R"
 			(at 2.54 1.92 0)
 			(layer "F.Fab")
@@
 			)
 		)
-		(property "Value" "220 Ohm"
+		(property "Value" "0 R"
 			(at 2.54 1.92 0)
 			(layer "F.Fab")
@@
 			)
 		)
-		(property "Value" "220 Ohm"
+		(property "Value" "0 R"
 			(at 2.54 1.92 0)
 			(layer "F.Fab")
@@
 			)
 		)
-		(property "Value" "220 Ohm"
+		(property "Value" "0 R"
 			(at 2.54 1.92 0)
 			(layer "F.Fab")
@@
 			)
 		)
-		(property "Value" "220 Ohm"
+		(property "Value" "0 R"
 			(at 2.54 1.92 0)
 			(layer "F.Fab")

Commit message: Add 28 switch-input debounce caps (100 nF) to the board
- Schematic: added C1-C28, one 100 nF cap from each switch input to GND,
  in parallel with the 10k pull-down (~1 ms RC debounce + noise filter on
  the long playfield leads). Enlarged the sheet to fit the cap bank. ERC at
  the benign baseline; all 28 netlist-verified across input<->GND.
- PCB: placed all 28 as 0805 SMD on the back, next to each pull-down (GND
  pad on the pour, input to the pull-down). 3D back render updated.
- BOM + guide + app schematic images updated (BOM total now $507.16, guide
  24 pages with a debounce-cap step). Synced to the live OneDrive KiCad.
Parts:
- added C1: 100nF, C_0805_2012Metric, B.Cu at (108.8, 60.9)
- added C10: 100nF, C_0805_2012Metric, B.Cu at (165.2, 51.4)
- added C11: 100nF, C_0805_2012Metric, B.Cu at (165.3, 45.9)
- added C12: 100nF, C_0805_2012Metric, B.Cu at (165.2, 40.4)
- added C13: 100nF, C_0805_2012Metric, B.Cu at (186.2, 60.9)
- added C14: 100nF, C_0805_2012Metric, B.Cu at (186.2, 66.4)
- added C15: 100nF, C_0805_2012Metric, B.Cu at (186.2, 71.9)
- added C16: 100nF, C_0805_2012Metric, B.Cu at (186.2, 77.4)
- added C17: 100nF, C_0805_2012Metric, B.Cu at (231.1, 77.2)
- added C18: 100nF, C_0805_2012Metric, B.Cu at (231.1, 72.2)
- added C19: 100nF, C_0805_2012Metric, B.Cu at (231.1, 67.2)
- added C2: 100nF, C_0805_2012Metric, B.Cu at (108.8, 66.4)
- added C20: 100nF, C_0805_2012Metric, B.Cu at (231.1, 62.2)
- added C21: 100nF, C_0805_2012Metric, B.Cu at (233.7, 55.2)
- added C22: 100nF, C_0805_2012Metric, B.Cu at (233.6, 50.2)
- added C23: 100nF, C_0805_2012Metric, B.Cu at (233.7, 45.2)
- added C24: 100nF, C_0805_2012Metric, B.Cu at (233.7, 40.7)
- added C25: 100nF, C_0805_2012Metric, B.Cu at (153.4, 109.2)
- added C26: 100nF, C_0805_2012Metric, B.Cu at (153.5, 103.7)
- added C27: 100nF, C_0805_2012Metric, B.Cu at (153.4, 98.2)
- added C28: 100nF, C_0805_2012Metric, B.Cu at (153.4, 92.7)
- added C3: 100nF, C_0805_2012Metric, B.Cu at (108.8, 71.9)
- added C4: 100nF, C_0805_2012Metric, B.Cu at (108.8, 77.4)
- added C5: 100nF, C_0805_2012Metric, B.Cu at (153.5, 77.4)
- added C6: 100nF, C_0805_2012Metric, B.Cu at (153.5, 72.4)
- added C7: 100nF, C_0805_2012Metric, B.Cu at (153.5, 66.4)
- added C8: 100nF, C_0805_2012Metric, B.Cu at (153.5, 61.4)
- added C9: 100nF, C_0805_2012Metric, B.Cu at (165.2, 56.4)
Routing:
- net GNDREF: track 589.1 -> 603.2 mm
- net Net-(SW9A-B): track 27.4 -> 29.7 mm
- net Net-(SW8A-B): track 26.4 -> 28.7 mm
- net Net-(SW3A-B): track 25.5 -> 27.8 mm
- net Net-(SW2A-B): track 21.2 -> 23.4 mm
- net Net-(SW23-1A-B): track 67.0 -> 69.2 mm
- net Net-(SW22A-B): track 27.2 -> 29.4 mm
- net Net-(SW21A-B): track 25.3 -> 27.5 mm
- net Net-(SW20A-B): track 25.1 -> 27.4 mm
- net Net-(SW1A-B): track 20.0 -> 22.2 mm
- net Net-(SW19A-B): track 21.8 -> 24.1 mm
- net Net-(SW18A-B): track 22.8 -> 25.1 mm
- net Net-(SW17A-B): track 22.6 -> 24.8 mm
- net Net-(SW16A-B): track 26.9 -> 29.1 mm
- net Net-(SW11A-B): track 31.0 -> 33.3 mm
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
Commit message: PCB: DRC 0/0 - drop 2 redundant GND tracks under the pour
The two long B.Cu GND tracks were already covered by the GND pour; with the
new cap pads in the pour they tripped a spurious cli-DRC clearance flag.
Removing them (pour keeps GND connected - 0 unconnected) makes the board
fully DRC clean.
Routing:
- net GNDREF: track 603.2 -> 547.3 mm
